Commit message: Add: - Naviagation package added. [Not Complete] - RL policy control added. [Complete]

File: robots/descriptions/go2_description/xacro/gazebo.xacro (robot description, xacro)
@@ -8,4 +8,19 @@
             <use_pose_vector_msg>true</use_pose_vector_msg>
             <update_frequency>10.0</update_frequency>
+        </plugin>
+    </gazebo>
+    <!-- Ground-truth base velocity, needed by the RL policy (controller:=model).
+         Its observation includes base linear velocity in the body frame, which nothing
+         else here publishes. The IMU gives orientation and angular velocity only, and
+         the PosePublisher above runs at 10 Hz with no twist. Ignition's OdometryPublisher
+         reports the twist in <robot_base_frame>, matching what the policy trained on.
+         Inert when running the CHAMP controller, since nothing subscribes. -->
+    <gazebo>
+        <plugin filename="ignition-gazebo-odometry-publisher-system" name="ignition::gazebo::systems::OdometryPublisher">
+            <odom_frame>odom_ground_truth</odom_frame>
+            <robot_base_frame>base_link</robot_base_frame>
+            <odom_publish_frequency>50</odom_publish_frequency>
+            <dimensions>3</dimensions>
+            <odom_topic>/odom_ground_truth</odom_topic>
         </plugin>
     </gazebo>

File: robots/descriptions/go2_description/xacro/laser.xacro (robot description, xacro)
@@ -31,5 +31,5 @@
             <visualize>false</visualize>
             <pose>0 0 0 0 0 0</pose>
-            <update_rate>50</update_rate>
+            <update_rate>10</update_rate>
             <topic>scan</topic>
             <ignition_frame_id>front_laser</ignition_frame_id>
@@ -37,5 +37,5 @@
             <scan>
                 <horizontal>
-                <samples>40</samples>
+                <samples>360</samples>
                 <resolution>1.000000</resolution>
                 <min_angle>0.000000</min_angle>
@@ -45,5 +45,5 @@
             <range>
                 <min>0.120000</min>
-                <max>3.5</max>
+                <max>12.0</max>
                 <resolution>0.015000</resolution>
             </range>

File: robots/descriptions/go2_description/xacro/leg.xacro (robot description, xacro)
@@ -189,4 +189,18 @@
             </joint>
         </ros2_control>
+        <!-- Foot contact sensor.
+             sdformat lumps the fixed-joint foot link into the lower leg, so the
+             sensor lives on ${name}_lower_leg_link and references the lumped
+             foot collision. champ's state estimator needs these contacts to
+             produce leg odometry; without them /odom never leaves the origin. -->
+        <gazebo reference="${name}_lower_leg_link">
+            <sensor name="${name}_foot_contact" type="contact">
+                <always_on>true</always_on>
+                <update_rate>50</update_rate>
+                <contact>
+                    <collision>${name}_lower_leg_link_fixed_joint_lump__${name}_foot_link_collision_1</collision>
+                </contact>
+            </sensor>
+        </gazebo>
         <!-- <xacro:leg_transmission name="${name}"/> -->
     </xacro:macro>
